File: karno65.kicad_pcb (KiCad board)
At the start: 2 copper layers, 154 parts, among them J1 AVR_ISP_6, J2 USB_OTG, SW1 GRV, SW10 9, SW11 0, SW12 MINS, SW13 EQL, SW14 SW_Push, SW15 SW_Push, SW16 TAB, SW17 Q, SW18 W, SW19 E, SW2 1, SW20 R, SW21 T, SW22 Y, SW23 U, SW24 I, SW25 O, SW26 P, SW27 LBRC, SW28 RBRC, SW29 BSLS, SW3 2, SW30 CAPS, SW31 A, SW32 S, SW33 D, SW34 F, SW35 G, SW36 H, SW37 J, SW38 K, SW39 L, SW4 3, SW40 SCLN, SW41 QUOT, SW42 ENT, SW43 LSFT, SW44 SW_Push, SW45 Z, SW46 X, SW47 C, SW48 V, SW49 B, SW5 4, SW50 N, SW51 M, SW52 COMM, SW53 DOT, SW54 SLSH, SW55 SW_Push, SW56 RSFT, SW57 LCTL, SW58 LGUI, SW59 LALT, SW6 5, SW60 SPC, SW61 RALT, SW62 RGUI, SW63 APP, SW64 RCTL, SW65 BSPC, SW7 6, SW8 7, SW9 8, U1 ATmega328-PU, Y1 16Mhz

Commit message: proto
Parts:
- added J3: ROWS, Connector_PinHeader_2.54mm:PinHeader_1x05_P2.54mm_Vertical, F.Cu at (73.7, 57.1)
- added J4: COLS, Connector_PinHeader_2.54mm:PinHeader_1x13_P2.54mm_Vertical, F.Cu at (81.3, 44.5)
- D1, D2, DS1, DS10, DS11, DS12, DS13, DS14, DS15, DS16, DS17, DS18, DS19, DS2, DS20, DS21, DS22, DS23, DS24, DS25, DS26, DS27, DS28, DS29, DS3, DS30, DS31, DS32, DS33, DS34, DS35, DS36, DS37, DS38, DS39, DS4, DS40, DS41, DS42, DS43, DS44, DS45, DS46, DS47, DS48, DS49, DS5, DS50, DS51, DS52, DS53, DS54, DS55, DS56, DS57, DS58, DS59, DS6, DS60, DS61, DS62, DS63, DS64, DS65, DS7, DS8, DS9: footprint Diode_THT:D_DO-35_SOD27_P5.08mm_Vertical_AnodeUp -> Diode_THT:D_DO-34_SOD68_P7.62mm_Horizontal
- F1: footprint Fuse:Fuse_Littelfuse_395Series -> Fuse:Fuse_BelFuse_0ZRE0005FF_L8.3mm_W3.8mm
- J2: footprint Connector_PinHeader_2.54mm:PinHeader_1x05_P2.54mm_Horizontal -> Connector_PinHeader_2.54mm:PinHeader_1x06_P2.54mm_Vertical
- R1, R2, R3, R4: footprint Resistor_THT:R_Axial_DIN0204_L3.6mm_D1.6mm_P5.08mm_Vertical -> Resistor_THT:R_Axial_DIN0204_L3.6mm_D1.6mm_P7.62mm_Horizontal
- moved C4 160.2 mm to (66.0, 22.9)
- moved SW_M1 158.9 mm to (48.3, 25.4)
- moved U1 158.0 mm to (106.7, 27.9)
- moved J1 157.9 mm to (48.3, 30.5)
- moved SW_M2 157.7 mm to (61.0, 25.4)
- moved C5 155.1 mm to (68.6, 22.9)
- moved C1 148.6 mm to (87.6, 21.6)
- moved Y1 145.3 mm to (78.7, 22.9), turned to 180 degrees
- moved R4 144.9 mm to (61.0, 30.5)
- moved C2 144.9 mm to (91.4, 25.4), turned to 90 degrees
- moved C3 142.3 mm to (94.0, 25.4), turned to 90 degrees
- moved R2 142.3 mm to (114.3, 25.4), turned to 0 degrees
- moved R3 139.7 mm to (114.3, 22.9), turned to 0 degrees
- moved R1 129.5 mm to (114.3, 27.9)
- moved D2 121.9 mm to (127.0, 30.5), turned to 90 degrees
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Connections:
- J2 pad 5: (no net) -> GND
Routing:
- net /COL4: track 0.00 -> 90.5 mm
- net GND: track 91.2 -> 154.8 mm
- net +5V: track 155.6 -> 104.8 mm
- net /ROW2: track 37.4 -> 81.3 mm
- net /ROW3: track 0.00 -> 41.9 mm
- net /COL1: track 0.00 -> 41.9 mm
- net /ROW0: track 36.4 -> 77.5 mm
- net /COL0: track 0.00 -> 40.4 mm
- net /ROW1: track 45.0 -> 82.5 mm
- net /COL2: track 33.2 -> 70.4 mm
- net /ROW4: track 0.00 -> 30.5 mm
- net /COL5: track 0.00 -> 26.2 mm
- net /COL10: track 0.00 -> 23.0 mm
- net /COL11: track 0.00 -> 21.9 mm
- net /RESET: track 77.1 -> 96.5 mm
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Other:
- board outline added: 101.6 x 44.5 mm
- net class Default: trace_width 1.2 -> 0.65
