File: karno65_controller_oneside.kicad_pcb (KiCad board)
At the start: 2 copper layers, 83.8 x 67.3 mm, 20 parts, among them J1 AVR_ISP_6, J2 USB_OTG, U1 ATmega328-PU, Y1 16Mhz

Commit message: one side
Parts:
- C4, C5: footprint Capacitor_THT:C_Disc_D3.0mm_W1.6mm_P2.50mm -> Capacitor_THT:C_Disc_D4.3mm_W1.9mm_P5.00mm
- moved REF** 48.3 mm to (58.4, 88.9)
- moved D1 40.6 mm to (177.8, 55.9)
- moved D2 40.6 mm to (177.8, 53.3)
- moved J2 40.6 mm to (190.5, 66.0)
- moved J1 22.3 mm to (81.3, 67.1), turned to 180 degrees
- moved SW_M1 15.5 mm to (132.1, 58.4), turned to 180 degrees
- moved R2 13.9 mm to (140.7, 57.9)
- moved R3 13.9 mm to (140.7, 55.4)
- moved R1 13.0 mm to (129.0, 68.6), turned to 90 degrees
- moved R4 11.9 mm to (125.5, 68.6), turned to 90 degrees
- moved SW_M2 11.0 mm to (72.8, 55.3)
- moved C4 10.8 mm to (89.5, 45.7), turned to 90 degrees
- moved C5 10.3 mm to (92.1, 45.7), turned to 90 degrees
- moved F1 8.59 mm to (133.6, 68.1), turned to 90 degrees
- moved C2 0.51 mm to (109.7, 55.9)
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Routing:
- net GND: track 155.1 -> 533.1 mm
- net /RESET: track 52.2 -> 110.3 mm, vias 2 -> 0
- net Net-(D2-Pad1): track 23.9 -> 73.6 mm
- net +5V: track 76.0 -> 44.5 mm, vias 2 -> 0
- net /COL2: track 98.0 -> 68.9 mm
- net Net-(D1-Pad1): track 35.0 -> 62.8 mm
- net /ROW1: track 30.5 -> 7.61 mm
- net /ROW0: track 38.2 -> 20.5 mm, vias 2 -> 0
- net /COL11: track 43.0 -> 25.2 mm
- net /ROW2: track 46.9 -> 31.7 mm, vias 2 -> 0
- net /USB_D+: track 16.3 -> 31.0 mm
- net /USB_D-: track 19.9 -> 32.7 mm
- net /COL1: track 61.0 -> 48.3 mm
- net /COL0: track 65.3 -> 55.2 mm
- net Net-(C4-Pad1): track 29.2 -> 20.9 mm
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Other:
- board outline removed
- net class Default: clearance 0.2 -> 0.4; trace_width 1.2 -> 0.5
- rule trace_clearance: 0.2 -> 0.4
