File: karno65_controller_satu_sisi.kicad_pcb (KiCad board)
At the start: 2 copper layers, 105.4 x 50.8 mm, 20 parts, among them J1 AVR_ISP_6, J2 USB_OTG, J3 ROWS, J4 COLS, U1 ATmega328-PU, Y1 16Mhz

Commit message: one side
Parts:
- removed J3: ROWS, Connector_PinHeader_2.54mm:PinHeader_1x05_P2.54mm_Vertical
- removed J4: COLS, Connector_PinHeader_2.54mm:PinHeader_1x13_P2.54mm_Vertical
- moved J1 10.2 mm to (86.4, 74.9), turned to 0 degrees
- moved R4 7.73 mm to (81.3, 72.4), turned to 270 degrees
Routing:
- net /ROW2: track 82.6 -> 0.00 mm
- net /COL3: track 68.6 -> 0.00 mm
- net /RESET: track 96.5 -> 159.8 mm
- net /COL1: track 43.5 -> 0.00 mm
- net /COL0: track 41.7 -> 0.00 mm
- net /COL2: track 69.1 -> 27.9 mm
- net /ROW3: track 43.2 -> 2.54 mm
- net /ROW1: track 83.8 -> 45.2 mm
- net /ROW4: track 33.0 -> 0.00 mm
- net /COL5: track 27.5 -> 0.00 mm
- net /COL4: track 27.0 -> 0.00 mm
- net /ROW0: track 78.7 -> 52.7 mm
- net GND: track 154.8 -> 132.5 mm
- net /COL12: track 17.8 -> 0.00 mm
- net +5V: track 104.8 -> 101.5 mm
Other:
- board outline removed

Commit message: one side
Parts:
- moved SW_M1 66.7 mm to (142.2, 78.1), turned to 90 degrees
- moved Y1 27.3 mm to (79.4, 66.7), turned to 270 degrees
- moved C5 21.6 mm to (74.9, 67.3)
- moved C3 21.3 mm to (142.9, 64.8), turned to 180 degrees
- moved C4 19.7 mm to (74.9, 71.1), turned to 270 degrees
- moved SW_M2 15.5 mm to (80.0, 81.3)
- moved R4 10.4 mm to (89.5, 78.7), turned to 90 degrees
- moved C2 10.3 mm to (128.9, 64.8), turned to 0 degrees
- moved J1 10.0 mm to (95.9, 78.1), turned to 180 degrees
- moved D1 8.51 mm to (166.0, 73.7)
- moved D2 8.51 mm to (163.4, 73.7)
- moved F1 8.51 mm to (152.0, 73.7)
- moved J2 8.51 mm to (171.1, 76.2)
- moved R1 8.51 mm to (150.7, 71.1)
- moved R2 8.51 mm to (150.7, 68.6)
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Routing:
- net +5V: track 101.5 -> 268.8 mm, vias 0 -> 4
- net /RESET: track 159.8 -> 64.5 mm, vias 0 -> 2
- net GND: track 132.5 -> 181.5 mm, vias 0 -> 4
- net /COL1: track 0.00 -> 39.9 mm
- net /ROW0: track 52.7 -> 17.6 mm
- net /COL0: track 0.00 -> 34.7 mm
- net /ROW2: track 0.00 -> 33.5 mm
- net /ROW3: track 2.54 -> 28.7 mm
- net /COL2: track 27.9 -> 53.6 mm
- net /ROW1: track 45.2 -> 20.8 mm
- net /COL3: track 0.00 -> 24.1 mm
- net Net-(C5-Pad1): track 26.5 -> 46.2 mm
- net Net-(C4-Pad1): track 25.5 -> 44.9 mm
- net /USB_D+: track 17.8 -> 26.2 mm
- net /COL10: track 25.0 -> 16.6 mm
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Other:
- net class Default: clearance 0.2 -> 0.24; via_dia 0.8 -> 0.6
- rule trace_clearance: 0.2 -> 0.24

Commit message: fix boot sw
Parts:
- moved Y1 5.75 mm to (73.6, 66.9), turned to 0 degrees
- moved C5 3.66 mm to (74.9, 71.0), turned to 180 degrees
- moved SW_M2 2.62 mm to (79.4, 78.7)
- moved C4 2.54 mm to (77.5, 71.0), turned to 0 degrees
Routing:
- net Net-(C5-Pad1): track 46.2 -> 50.6 mm
- net GND: track 181.5 -> 184.4 mm
- net Net-(C4-Pad1): track 44.9 -> 42.3 mm
- net +5V: track 268.8 -> 267.6 mm
- net /ROW2: track 33.5 -> 34.2 mm
- net /COL2: track 53.6 -> 52.9 mm

Commit message: via 0.9
Parts:
- moved Y1 153.9 mm to (222.9, 29.2)
- moved C4 153.9 mm to (226.7, 33.5)
- moved C5 153.9 mm to (224.2, 33.5)
- moved SW_M2 153.7 mm to (228.6, 41.9)
- moved J1 153.1 mm to (244.5, 41.3)
- moved R4 152.9 mm to (238.1, 42.5)
- moved C2 152.5 mm to (276.9, 27.9)
- moved C3 152.5 mm to (290.8, 27.9)
- moved U1 152.5 mm to (282.6, 34.3)
- moved C1 152.3 mm to (267.3, 29.8)
- moved SW_M1 151.9 mm to (289.6, 41.3)
- moved F1 150.6 mm to (298.1, 36.8)
- moved R1 150.6 mm to (296.8, 34.3)
- moved R2 150.6 mm to (296.8, 31.8)
- moved R3 150.6 mm to (296.8, 29.2)
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Routing:
- net +5V: track 267.6 -> 257.6 mm
- net Net-(F1-Pad2): track 19.4 -> 11.7 mm
- net Net-(D2-Pad1): track 27.0 -> 19.8 mm
- net Net-(D1-Pad1): track 16.3 -> 12.1 mm
- net /COL3: track 24.1 -> 21.0 mm
- net /ROW1: track 20.8 -> 18.0 mm
- net /RESET: track 64.5 -> 62.1 mm
- net GND: track 184.4 -> 182.4 mm
- net /USB_D+: track 26.2 -> 24.3 mm
- net Net-(C4-Pad1): track 42.3 -> 40.6 mm
- net /USB_D-: track 28.8 -> 27.2 mm
- net /ROW0: track 17.6 -> 16.1 mm
- net Net-(C5-Pad1): track 50.6 -> 49.1 mm
- net /COL11: track 16.1 -> 14.8 mm
- net /ROW3: track 28.7 -> 27.5 mm
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Other:
- net class Default: clearance 0.24 -> 0.3; via_dia 0.6 -> 1.6; via_drill 0.4 -> 1
- rule trace_clearance: 0.24 -> 0.3
